File: Octal Display board/OctalBusDisplay/OctalBusDisplay.kicad_pcb (KiCad board)
At the start: 2 copper layers, 100 x 51 mm, 18 parts, among them IC1 TIL311, IC10 TIL311, IC11 TIL311, IC12 TIL311, IC13 TIL311, IC14 TIL311, IC2 TIL311, IC3 TIL311, IC4 TIL311, IC5 TIL311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

Commit message: Added 16x16 dotmatrix display PCB and test code
Connections:
- IC1 pad 10: GND -> unconnected-(IC1-RIGHT_DOT-Pad10)
- IC1 pad 4: GND -> unconnected-(IC1-LEFT_DOT-Pad4)
- IC10 pad 10: GND -> unconnected-(IC10-RIGHT_DOT-Pad10)
- IC10 pad 4: GND -> unconnected-(IC10-LEFT_DOT-Pad4)
- IC11 pad 10: GND -> unconnected-(IC11-RIGHT_DOT-Pad10)
- IC11 pad 4: GND -> unconnected-(IC11-LEFT_DOT-Pad4)
- IC12 pad 10: GND -> unconnected-(IC12-RIGHT_DOT-Pad10)
- IC12 pad 4: GND -> unconnected-(IC12-LEFT_DOT-Pad4)
- IC13 pad 10: GND -> unconnected-(IC13-RIGHT_DOT-Pad10)
- IC13 pad 4: GND -> unconnected-(IC13-LEFT_DOT-Pad4)
- IC14 pad 10: GND -> unconnected-(IC14-RIGHT_DOT-Pad10)
- IC14 pad 4: GND -> unconnected-(IC14-LEFT_DOT-Pad4)
- IC2 pad 10: GND -> unconnected-(IC2-RIGHT_DOT-Pad10)
- IC2 pad 4: GND -> unconnected-(IC2-LEFT_DOT-Pad4)
- IC3 pad 10: GND -> unconnected-(IC3-RIGHT_DOT-Pad10)
- IC3 pad 4: GND -> unconnected-(IC3-LEFT_DOT-Pad4)
- IC4 pad 10: GND -> unconnected-(IC4-RIGHT_DOT-Pad10)
- IC4 pad 4: GND -> unconnected-(IC4-LEFT_DOT-Pad4)
- IC5 pad 10: GND -> unconnected-(IC5-RIGHT_DOT-Pad10)
- IC5 pad 4: GND -> unconnected-(IC5-LEFT_DOT-Pad4)
- IC6 pad 10: GND -> unconnected-(IC6-RIGHT_DOT-Pad10)
- IC6 pad 4: GND -> unconnected-(IC6-LEFT_DOT-Pad4)
- IC7 pad 10: GND -> unconnected-(IC7-RIGHT_DOT-Pad10)
- IC7 pad 4: GND -> unconnected-(IC7-LEFT_DOT-Pad4)
- IC8 pad 10: GND -> unconnected-(IC8-RIGHT_DOT-Pad10)
- IC8 pad 4: GND -> unconnected-(IC8-LEFT_DOT-Pad4)
- IC9 pad 10: GND -> unconnected-(IC9-RIGHT_DOT-Pad10)
- IC9 pad 4: GND -> unconnected-(IC9-LEFT_DOT-Pad4)
Routing:
- net GND: track 77.3 -> 36.0 mm, vias 2 -> 1
- net unconnected-(IC5-LEFT_DOT-Pad4): track 0.00 -> 7.52 mm, vias 0 -> 1
- net /LA2: track 38.5 -> 37.6 mm
