File: Display 16x16/16x16display.kicad_pcb (KiCad board)
At the start: 2 copper layers, 100 x 100 mm, 41 parts, among them J1 86093967113745ELF, U1 7130LA55PDGI, U10 SN74AHCT240DWR, U2 GAL16V8, U3 GAL16V8, U4 74ahc1G14dckr, U5 74HCT238, U6 74HCT238, U7 74HCT238, U8 74HCT238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

Commit message: Update with correct chips (no change to PCB)
Parts:
- U10: value SN74AHCT240DWR -> SN74AHCT244DWR
- U5, U6, U7, U8: value 74HCT238 -> 74HC138
